File: christmas tree.kicad_pcb (KiCad board)
At the start: 2 copper layers, 50 x 54.2 mm, 0 parts

Commit message: added components, and deco
Parts:
- added BAT1: BS-7, digikey-footprints:Battery_Holder_Coin_2032_BS-7, F.Cu at (152.6, 121.5)
- added D1: LED, LED_THT:LED_D5.0mm, B.Cu at (147.4, 136.4)
- added D2: LED, LED_THT:LED_D5.0mm, B.Cu at (166.5, 131.6)
- added D3: LED, LED_THT:LED_D5.0mm, B.Cu at (167.9, 115.8)
- added D4: LED, LED_THT:LED_D5.0mm, B.Cu at (165.5, 102.9)
- added D5: LED, LED_THT:LED_D5.0mm, B.Cu at (157.6, 104.4)
- added D6: LED, LED_THT:LED_D5.0mm, B.Cu at (156.2, 115.3)
- added D7: LED, LED_THT:LED_D5.0mm, B.Cu at (154.3, 128.0)
- added SW1: SW_SPST, digikey-footprints:Switch_Slide_11.6x4mm_EG1218, F.Cu at (174.6, 138.9)
Routing:
- net Net-(D1-Pad2): track 0.00 -> 25.7 mm
- net Net-(BAT1-PadPos): track 0.00 -> 19.2 mm
- net Net-(D1-Pad1): track 0.00 -> 18.5 mm
- net Net-(D2-Pad1): track 0.00 -> 16.2 mm
- net Net-(D6-Pad1): track 0.00 -> 13.0 mm
- net Net-(D3-Pad1): track 0.00 -> 11.4 mm
- net Net-(D5-Pad1): track 0.00 -> 8.96 mm
- net Net-(D4-Pad1): track 0.00 -> 8.29 mm
- net Net-(BAT1-PadNeg): track 0.00 -> 7.16 mm
Other:
- board size 50 x 54.2 mm -> 50 x 62.4 mm
