File: christmas tree.kicad_pcb (KiCad board)
At the start: 2 copper layers, 50 x 62.4 mm, 9 parts, among them SW1 SW_SPST

Commit message: retraced the circuit
still don't know if this will work
Parts:
- removed D5: LED, LED_THT:LED_D5.0mm
- added Dr: LED, LED_THT:LED_D5.0mm, B.Cu at (168.0, 129.8)
- moved D1 37.9 mm to (164.7, 102.7), turned to 90 degrees
- moved D6 27.2 mm to (145.2, 140.2)
- moved D3 18.2 mm to (155.4, 102.6), turned to 90 degrees
- moved D2 16.8 mm to (167.8, 114.8)
- moved D4 13.6 mm to (157.2, 113.7), turned to 180 degrees
- moved D7 2.24 mm to (155.8, 129.7), turned to 90 degrees
- moved SW1 1.81 mm to (176.3, 139.6)
- moved BAT1 0.19 mm to (152.8, 121.5)
Connections:
- D1 pad 1: Net-(D1-Pad1) -> Net-(BAT1-PadNeg)
- D1 pad 2: Net-(D1-Pad2) -> Net-(D2-Pad2)
- D2 pad 1: Net-(D2-Pad1) -> Net-(BAT1-PadNeg)
- D2 pad 2: Net-(D1-Pad1) -> Net-(D2-Pad2)
- D3 pad 1: Net-(D3-Pad1) -> Net-(BAT1-PadNeg)
- D3 pad 2: Net-(D2-Pad1) -> Net-(D2-Pad2)
- D4 pad 1: Net-(D4-Pad1) -> Net-(BAT1-PadNeg)
- D4 pad 2: Net-(D3-Pad1) -> Net-(D2-Pad2)
- D6 pad 1: Net-(D6-Pad1) -> Net-(BAT1-PadNeg)
- D6 pad 2: Net-(D5-Pad1) -> Net-(D2-Pad2)
- D7 pad 2: Net-(D6-Pad1) -> Net-(D2-Pad2)
- SW1 pad 2: Net-(D1-Pad2) -> Net-(D2-Pad2)
Routing:
- net Net-(D2-Pad2): track 0.00 -> 106.1 mm
- net Net-(BAT1-PadNeg): track 7.16 -> 98.9 mm
- net Net-(D1-Pad2): track 25.7 -> 0.00 mm
- net Net-(D1-Pad1): track 18.5 -> 0.00 mm
- net Net-(D2-Pad1): track 16.2 -> 0.00 mm
- net Net-(D6-Pad1): track 13.0 -> 0.00 mm
- net Net-(D3-Pad1): track 11.4 -> 0.00 mm
- net Net-(D5-Pad1): track 8.96 -> 0.00 mm
- net Net-(D4-Pad1): track 8.29 -> 0.00 mm
- net Net-(BAT1-PadPos): track 19.2 -> 20.6 mm

Commit message: Sized switch
Routing:
- net Net-(D2-Pad2): track 106.1 -> 104.3 mm
