File: christmas tree.kicad_sch (KiCad schematic)
At the start: 8 parts

Commit message: added components, and deco
Parts:
- added D7: LED, LED_THT:LED_D5.0mm, symbol Device:LED
- BAT1: value (none) -> BS-7; footprint (none) -> digikey-footprints:Battery_Holder_Coin_2032_BS-7
- D1, D2, D3, D4, D5, D6: value (none) -> LED; footprint (none) -> LED_THT:LED_D5.0mm
- SW1: value (none) -> SW_SPST; footprint (none) -> digikey-footprints:Switch_Slide_11.6x4mm_EG1218
Connections:
- net at BAT1.Neg: now also D7.1 (K); no longer D6.1 (K)
- new net: D6.1 (K), D7.2 (A)
Changed lines of the file:
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@@
     (stroke (width 0) (type default) (color 0 0 0 0))
   )
-  (wire (pts (xy 176.53 43.942) (xy 176.53 81.026))
+  (wire (pts (xy 176.53 43.942) (xy 176.53 47.498))
+    (stroke (width 0) (type default) (color 0 0 0 0))
+  )
+  (wire (pts (xy 176.53 55.118) (xy 176.53 81.026))
     (stroke (width 0) (type default) (color 0 0 0 0))
   )
@@
     (in_bom yes) (on_board yes) (fields_autoplaced)
     (property "Reference" "D2" (id 0) (at 128.0795 36.83 0))
-    (property "Value" "" (id 1) (at 128.0795 39.37 0))
-    (property "Footprint" "" (id 2) (at 126.492 43.942 0)
+    (property "Value" "LED" (id 1) (at 128.0795 39.37 0))
+    (property "Footprint" "LED_THT:LED_D5.0mm" (id 2) (at 126.492 43.942 0)
       (effects (font (size 1.27 1.27)) hide)
     )
@@
     (in_bom yes) (on_board yes) (fields_autoplaced)
     (property "Reference" "D4" (id 0) (at 152.4635 36.83 0))
-    (property "Value" "" (id 1) (at 152.4635 39.37 0))
-    (property "Footprint" "" (id 2) (at 150.876 43.942 0)
+    (property "Value" "LED" (id 1) (at 152.4635 39.37 0))
+    (property "Footprint" "LED_THT:LED_D5.0mm" (id 2) (at 150.876 43.942 0)
       (effects (font (size 1.27 1.27)) hide)
     )
@@
     (in_bom yes) (on_board yes) (fields_autoplaced)
     (property "Reference" "D5" (id 0) (at 163.8935 36.83 0))
-    (property "Value" "" (id 1) (at 163.8935 39.37 0))
-    (property "Footprint" "" (id 2) (at 162.306 43.942 0)
+    (property "Value" "LED" (id 1) (at 163.8935 39.37 0))
+    (property "Footprint" "LED_THT:LED_D5.0mm" (id 2) (at 162.306 43.942 0)
       (effects (font (size 1.27 1.27)) hide)
     )
@@
     (in_bom yes) (on_board yes) (fields_autoplaced)
     (property "Reference" "D3" (id 0) (at 140.0175 36.83 0))
-    (property "Value" "" (id 1) (at 140.0175 39.37 0))
-    (property "Footprint" "" (id 2) (at 138.43 43.942 0)
+    (property "Value" "LED" (id 1) (at 140.0175 39.37 0))
+    (property "Footprint" "LED_THT:LED_D5.0mm" (id 2) (at 138.43 43.942 0)
       (effects (font (size 1.27 1.27)) hide)
     )
@@
     (in_bom yes) (on_board yes) (fields_autoplaced)
     (property "Reference" "SW1" (id 0) (at 92.71 55.88 0))
-    (property "Value" "" (id 1) (at 92.71 58.42 0))
-    (property "Footprint" "" (id 2) (at 92.71 62.484 0)
+    (property "Value" "SW_SPST" (id 1) (at 92.71 58.42 0))
+    (property "Footprint" "digikey-footprints:Switch_Slide_11.6x4mm_EG1218" (id 2) (at 92.71 62.484 0)
       (effects (font (size 1.27 1.27)) hide)
     )
@@
       (effects (font (size 1.524 1.524)) (justify left))
     )
-    (property "Value" "" (id 1) (at 91.44 78.105 0)
+    (property "Value" "BS-7" (id 1) (at 91.44 78.105 0)
       (effects (font (size 1.524 1.524)) (justify left))
     )
-    (property "Footprint" "" (id 2) (at 92.71 70.866 0)
+    (property "Footprint" "digikey-footprints:Battery_Holder_Coin_2032_BS-7" (id 2) (at 92.71 70.866 0)
       (effects (font (size 1.524 1.524)) (justify left) hide)
     )
@@
     (in_bom yes) (on_board yes) (fields_autoplaced)
     (property "Reference" "D1" (id 0) (at 116.1415 36.83 0))
-    (property "Value" "" (id 1) (at 116.1415 39.37 0))
-    (property "Footprint" "" (id 2) (at 114.554 43.942 0)
+    (property "Value" "LED" (id 1) (at 116.1415 39.37 0))
+    (property "Footprint" "LED_THT:LED_D5.0mm" (id 2) (at 114.554 43.942 0)
       (effects (font (size 1.27 1.27)) hide)
     )
@@
     (in_bom yes) (on_board yes) (fields_autoplaced)
     (property "Reference" "D6" (id 0) (at 174.3075 36.83 0))
-    (property "Value" "" (id 1) (at 174.3075 39.37 0))
-    (property "Footprint" "" (id 2) (at 172.72 43.942 0)
+    (property "Value" "LED" (id 1) (at 174.3075 39.37 0))
+    (property "Footprint" "LED_THT:LED_D5.0mm" (id 2) (at 172.72 43.942 0)
       (effects (font (size 1.27 1.27)) hide)
     )
     (property "Datasheet" "~" (id 3) (at 172.72 43.942 0)
+      (effects (font (size 1.27 1.27)) hide)
+    )
+    (pin "1")
+    (pin "2")
+  )
+  (symbol (lib_id "Device:LED") (at 176.53 51.308 90) (unit 1)
+    (in_bom yes) (on_board yes) (fields_autoplaced)
+    (property "Reference" "D7" (id 0) (at 180.34 51.6254 90)
+      (effects (font (size 1.27 1.27)) (justify right))
+    )
+    (property "Value" "LED" (id 1) (at 180.34 54.1654 90)
+      (effects (font (size 1.27 1.27)) (justify right))
+    )
+    (property "Footprint" "LED_THT:LED_D5.0mm" (id 2) (at 176.53 51.308 0)
+      (effects (font (size 1.27 1.27)) hide)
+    )
+    (property "Datasheet" "~" (id 3) (at 176.53 51.308 0)
       (effects (font (size 1.27 1.27)) hide)
     )
@@
       (reference "D6") (unit 1) (value "LED") (footprint "LED_THT:LED_D5.0mm")
     )
+    (path "/9c3944cd-af5e-4177-a216-36500543154a"
+      (reference "D7") (unit 1) (value "LED") (footprint "LED_THT:LED_D5.0mm")
+    )
     (path "/4579c54c-b265-4aa5-9a87-4007d2b1ecef"

Commit message: retraced the circuit
still don't know if this will work
Connections:
- net at D2.1 (K): now also BAT1.Neg, D1.1 (K), D3.1 (K), D4.1 (K), D5.1 (K), D6.1 (K), D7.1 (K); no longer D3.2 (A)
- net at D2.2 (A): now also D1.2 (A), D3.2 (A), D4.2 (A), D5.2 (A), D6.2 (A), D7.2 (A), SW1.2 (B); no longer D1.1 (K)
Other:
- moved on the sheet: BAT1, D1, D2, D3, D4, D5, D6, D7, SW1
